File: resources/KiCad/DuelWithBanjos/Battery_Power.kicad_sch (KiCad schematic)
At the start: 6 parts, among them J1 Conn_01x03_Pin, J2 Conn_01x03_Socket, SW1 SW_SPST

Commit message: pin assignments and schematic first cut
Connections:
- net at SW1.~ (B): now also J1.1 (Pin_1)
Changed lines of the file:
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@@
 	(title_block
 		(title "DuelWithBanjos")
-		(date "2025-03-14")
+		(date "2025-03-16")
 		(rev "Rev 0.9")
 		(company "https://github.com/Mark-MDO47")

Commit message: update schematic
Connections:
- net at SW1.~ (B): now also J1.1 (Pin_1)
Changed lines of the file:
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@@
 	(title_block
 		(title "DuelWithBanjos")
-		(date "2025-03-16")
+		(date "2025-03-19")
 		(rev "Rev 0.9")
 		(company "https://github.com/Mark-MDO47")

Commit message: add connectors for skeletons, move deck chairs around
Connections:
- net at SW1.~ (B): now also J1.1 (Pin_1)
Changed lines of the file:
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@@
 	(title_block
 		(title "DuelWithBanjos")
-		(date "2025-03-19")
+		(date "2025-04-10")
 		(rev "Rev 0.9")
 		(company "https://github.com/Mark-MDO47")

Commit message: move pins farther apart
Connections:
- net at SW1.~ (B): now also J1.1 (Pin_1)
Changed lines of the file:
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@@
 	(title_block
 		(title "DuelWithBanjos")
-		(date "2025-04-10")
+		(date "2025-04-13")
 		(rev "Rev 0.9")
 		(company "https://github.com/Mark-MDO47")

Commit message: KiCad V9.0.1
Connections:
- net at SW1.~ (B): now also J1.1 (Pin_1)
Changed lines of the file:
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@@
 (kicad_sch
-	(version 20231120)
+	(version 20250114)
 	(generator "eeschema")
-	(generator_version "8.0")
+	(generator_version "9.0")
 	(paper "A4")
 	(title_block
 		(title "DuelWithBanjos")
-		(date "2025-04-13")
+		(date "2025-05-08")
 		(rev "Rev 0.9")
 		(company "https://github.com/Mark-MDO47")
 	)
+	(text "Red"
+		(exclude_from_sim no)
+		(at 80.264 68.58 0)
+		(effects
+			(font
+				(size 1.27 1.27)
+			)
+		)
+	)
+	(text "JST"
+		(exclude_from_sim no)
+		(at 81.534 86.614 0)
+		(effects
+			(font
+				(size 3 3)
+			)
+		)
+	)
+	(text "White"
+		(exclude_from_sim no)
+		(at 81.026 73.66 0)
+		(effects
+			(font
+				(size 1.27 1.27)
+			)
+		)
+	)
+	(text "3.8V"
+		(exclude_from_sim no)
+		(at 33.02 99.06 0)
+		(effects
+			(font
+				(size 1.27 1.27)
+				(bold yes)
+			)
+			(justify right bottom)
+		)
+	)
+	(text "3.8V"
+		(exclude_from_sim no)
+		(at 33.02 81.28 0)
+		(effects
+			(font
+				(size 1.27 1.27)
+				(bold yes)
+			)
+			(justify right bottom)
+		)
+	)
+	(text "3.8V"
+		(exclude_from_sim no)
+		(at 33.02 63.5 0)
+		(effects
+			(font
+				(size 1.27 1.27)
+				(bold yes)
+			)
+			(justify right bottom)
+		)
+	)
 	(wire
 		(pts
@@
 			(width 0)
 			(type default)
-		)
-	)
-	(text "Red"
-		(exclude_from_sim no)
-		(at 80.264 68.58 0)
-		(effects
-			(font
-				(size 1.27 1.27)
-			)
-		)
-	)
-	(text "JST"
-		(exclude_from_sim no)
-		(at 81.534 86.614 0)
-		(effects
-			(font
-				(size 3 3)
-			)
-		)
-	)
-	(text "White"
-		(exclude_from_sim no)
-		(at 81.026 73.66 0)
-		(effects
-			(font
-				(size 1.27 1.27)
-			)
-		)
-	)
-	(text "3.8V"
-		(exclude_from_sim no)
-		(at 33.02 99.06 0)
-		(effects
-			(font
-				(size 1.27 1.27)
-				(bold yes)
-			)
-			(justify right bottom)
-		)
-	)
-	(text "3.8V"
-		(exclude_from_sim no)
-		(at 33.02 81.28 0)
-		(effects
-			(font
-				(size 1.27 1.27)
-				(bold yes)
-			)
-			(justify right bottom)
-		)
-	)
-	(text "3.8V"
-		(exclude_from_sim no)
-		(at 33.02 63.5 0)
-		(effects
-			(font
-				(size 1.27 1.27)
-				(bold yes)
-			)
-			(justify right bottom)
 		)
 	)
@@
 		(shape output)
 		(at 205.74 68.58 0)
-		(fields_autoplaced yes)
 		(effects
 			(font
@@
 		(shape output)
 		(at 205.74 78.74 0)
-		(fields_autoplaced yes)
-		(effects
-			(font
+		(effects
+			(font

Commit message: DS3502_digi_pot does not have enough current capacity on wiper
Connections:
- net at SW1.~ (B): now also J1.1 (Pin_1)
Changed lines of the file:
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@@
 	(title_block
 		(title "DuelWithBanjos")
-		(date "2025-05-08")
+		(date "2025-05-30")
 		(rev "Rev 0.9")
 		(company "https://github.com/Mark-MDO47")
